File: 0-35V 0-3A/kicad/power_supply_35V_3A.kicad_pcb (KiCad board)
At the start: 2 copper layers, 138 x 100 mm, 130 parts, among them J1 220VAC, J10 OUT_NEGATIVE, J11 LED_PG_5VA, J12 LED_PG_3V3, J13 Fixed outputs, J14 LED_PG_5VB, J2 TRANSISTORS, J3 VOLTAGE_POT, J4 CURRENT_POT, J5 33VAC_4A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

Commit message: Fix PCB ground planes
Parts:
- removed JP3, JP5, JP8, JP9: GND_CONNECT, Jumper:SolderJumper-2_P1.3mm_Open_Pad1.0x1.5mm
- removed the JP4 at (105.9, -27.1)
- added JP2: GND_CONNECT, Jumper:SolderJumper-2_P1.3mm_Open_Pad1.0x1.5mm, F.Cu at (122.9, -13.8)
- added JP2: GND_CONNECT, Jumper:SolderJumper-2_P1.3mm_Open_Pad1.0x1.5mm, F.Cu at (125.0, -11.7)
- added JP4: GND_CONNECT, Jumper:SolderJumper-2_P1.3mm_Open_Pad1.0x1.5mm, B.Cu at (116.5, -20.5)
- added JP4: GND_CONNECT, Jumper:SolderJumper-2_P1.3mm_Open_Pad1.0x1.5mm, B.Cu at (104.5, -31.2)
- added JP4: GND_CONNECT, Jumper:SolderJumper-2_P1.3mm_Open_Pad1.0x1.5mm, B.Cu at (100.0, -35.7)
- added JP4: GND_CONNECT, Jumper:SolderJumper-2_P1.3mm_Open_Pad1.0x1.5mm, B.Cu at (109.4, -26.6)
- added JPe: GND_CONNECT, Jumper:SolderJumper-2_P1.3mm_Open_Pad1.0x1.5mm, B.Cu at (126.0, -10.7)
- added REF**: GND to chassis, TestPoint:TestPoint_THTPad_4.0x4.0mm_Drill2.0mm, F.Cu at (134.7, -10.7)
- moved C13 11.8 mm to (129.0, -20.6), turned to 270 degrees
- moved J10 11.8 mm to (131.7, -28.7)
- moved R25 11.4 mm to (126.9, -20.6), turned to 270 degrees
- moved J9 9.38 mm to (131.7, -18.6)
- moved TP6 9.25 mm to (109.5, -14.4)
- moved C15 8.27 mm to (122.7, -22.6), turned to 90 degrees
- moved R26 8.22 mm to (129.2, -27.6), turned to 270 degrees
- moved C14 3.29 mm to (135.5, -23.6), turned to 180 degrees
Connections:
- J9 pad 1: Net-(C13-Pad1) -> GNDA
- J9 pad 2: GNDA -> Net-(C13-Pad1)
Routing:
- net GNDA: track 239.6 -> 274.7 mm
- net Net-(J10-Pad1): track 108.6 -> 87.6 mm
- net GND: track 99.2 -> 90.8 mm, vias 163 -> 87
- net Net-(J14-Pad1): track 46.0 -> 43.4 mm
- net Net-(J14-Pad2): track 55.8 -> 53.2 mm
- net Net-(C13-Pad1): track 59.5 -> 57.1 mm
- net +5V_A: track 39.0 -> 37.7 mm, vias 1 -> 0
- net +12V: track 167.3 -> 166.2 mm
- net GNDB: vias 71 -> 72
