File: 0-35V 0-3A/kicad/regulated_supply.sch (KiCad schematic (older format))
At the start: 73 parts, among them J10 OUT_NEGATIVE, J2 TRANSISTORS, J3 VOLTAGE_POT, J4 CURRENT_POT, J5 33VAC_4A, J6 AMMETER_2V_RANGE, J7 VMETER_200MV_RANGE, J8 LED_CURRENT_LIMIT, J9 OUT_POSITIVE, Q1 BD911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

Commit message: Fix PCB ground planes
Connections:
- net GNDA: now also J9.1 (Pin_1); no longer J9.2 (Pin_2)
- net at C13.1, C14.2, C15.1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: now also J9.2 (Pin_2); no longer J9.1 (Pin_1)
Other:
- moved on the sheet: J9
Changed lines of the file:
@@
 L Connector:Screw_Terminal_01x02 J?
 U 1 1 609D01BF
-P 11000 3200
+P 11050 3300
 AR Path="/609D01BF" Ref="J?"  Part="1"
 AR Path="/60972626/609D01BF" Ref="J9"  Part="1"
-F 0 "J9" H 11000 3000 50  0000 C CNN
-F 1 "OUT_POSITIVE" V 11100 3250 50  0000 C CNN
-F 2 "TerminalBlock_RND:TerminalBlock_RND_205-00001_1x02_P5.00mm_Horizontal" H 11000 3200 50  0001 C CNN
-F 3 "~" H 11000 3200 50  0001 C CNN
-	1    11000 3200
-	1    0    0    -1
+F 0 "J9" H 11050 3100 50  0000 C CNN
+F 1 "OUT_POSITIVE" V 11150 3350 50  0000 C CNN
+F 2 "TerminalBlock_RND:TerminalBlock_RND_205-00001_1x02_P5.00mm_Horizontal" H 11050 3300 50  0001 C CNN
+F 3 "~" H 11050 3300 50  0001 C CNN
+	1    11050 3300
+	1    0    0    1
 $EndComp
 $Comp
@@
 Wire Wire Line
 	10500 3200 10500 3000
-Wire Wire Line
-	10500 3200 10800 3200
 Connection ~ 10500 3000
 Wire Wire Line
@@
 Wire Wire Line
 	10500 3200 10250 3200
-Connection ~ 10500 3200
 Wire Wire Line
 	10250 3200 10050 3200
@@
 Wire Wire Line
 	10250 3500 10450 3500
-Wire Wire Line
-	10800 3500 10800 3300
 Connection ~ 10250 3500
 Text GLabel 10450 3700 3    50   Input ~ 0
@@
 	1    0    0    -1
 $EndComp
+Wire Wire Line
+	10850 3200 10500 3200
+Connection ~ 10500 3200
+Wire Wire Line
+	10800 3500 10800 3300
+Wire Wire Line
+	10800 3300 10850 3300
 $EndSCHEMATC
